File: belliot.kicad_pcb (KiCad board)
At the start: 2 copper layers, 41 x 71 mm, 22 parts, among them J1 Screw_Terminal_01x02, J2 Screw_Terminal_01x02, J3 LED, J4 SWITCH, K1 G6K-2, K2 G6K-2, Q1 IRLML2502, Q2 IRLML2502, U1 WeMos_D1_mini, U2 VOS628A

Commit message: some improvements
Parts:
- removed J1, J2: Screw_Terminal_01x02, TerminalBlock:TerminalBlock_bornier-2_P5.08mm
- removed R2: 3k9, Resistor_SMD:R_0805_2012Metric_Pad1.20x1.40mm_HandSolder
- added J5: Screw_Terminal_01x04, TerminalBlock_Phoenix:TerminalBlock_Phoenix_MKDS-1,5-4-5.08_1x04_P5.08mm_Horizontal, F.Cu at (127.3, 88.4)
- H1, H2, H3, H4: footprint MountingHole:MountingHole_2.5mm -> MountingHole:MountingHole_2.7mm
- J3, J4: footprint TestPoint:TestPoint_2Pads_Pitch5.08mm_Drill1.3mm -> Connector_PinHeader_2.54mm:PinHeader_1x02_P2.54mm_Vertical
- K1, K2: value G6K-2 -> G6K-2F-Y
- moved R4 9.77 mm to (139.2, 99.3), turned to 270 degrees
- moved J4 3.81 mm to (136.4, 122.9), turned to 90 degrees
- moved R3 2.03 mm to (139.2, 90.4)
- moved J3 1.30 mm to (136.4, 119.1), turned to 90 degrees
Connections:
- U1 pad 11: Net-(J4-Pad1) -> Net-(U1-Pad11)
- U1 pad 3: Net-(R4-Pad1) -> Net-(U1-Pad3)
- U1 pad 4: Net-(U1-Pad4) -> Net-(R4-Pad1)
- U1 pad 5: Net-(U1-Pad5) -> Net-(J4-Pad1)
Routing:
- net +5V: track 108.1 -> 87.8 mm, vias 0 -> 1
- net +3V3: track 21.8 -> 7.68 mm, vias 1 -> 0
- net 7: track 53.7 -> 51.5 mm
- net Net-(R3-Pad1): track 5.04 -> 3.06 mm
- net Net-(J4-Pad1): track 33.3 -> 31.5 mm
- net c: track 31.8 -> 32.4 mm
- net Net-(J3-Pad1): track 6.15 -> 5.64 mm
- net Net-(R4-Pad1): track 13.1 -> 13.3 mm, vias 1 -> 0
Other:
- board size 41 x 71 mm -> 46 x 71 mm
- board text added: "Belliot 1.1"
- board text removed: "Belliot 1.0"
